File: Synth/wavefolder.kicad_sch (KiCad schematic)
At the start: 19 parts, among them Q1 PNP, Q2 NPN, Q3 PNP, Q4 NPN, U3 LM321, U4 LM321, U5 LM321

Commit message: removed mixer
Connections:
- net V_DD is gone; now on net +12V: U3.5 (V+)
- net +12V: now also U5.5 (V+)
- net GND: now also U5.2 (V-)
Changed lines of the file:
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@@
-    )
-  )
-  (global_label "V_DD" (shape input) (at 96.52 79.375 90) (fields_autoplaced)
-    (effects (font (size 1.27 1.27)) (justify left))
-    (property "Intersheetrefs" "${INTERSHEET_REFS}" (at 96.52 71.7936 90)
-      (effects (font (size 1.27 1.27)) (justify left) hide)
     )
   )
@@
     )
   )
+  (symbol (lib_id "power:GND") (at 192.405 89.535 0) (unit 1)
+    (in_bom yes) (on_board yes) (dnp no) (fields_autoplaced)
+    (property "Reference" "#PWR05" (at 192.405 95.885 0)
+      (effects (font (size 1.27 1.27)) hide)
+    )
+    (property "Value" "GND" (at 192.405 94.869 0)
+      (effects (font (size 1.27 1.27)))
+    )
+    (property "Footprint" "" (at 192.405 89.535 0)
+      (effects (font (size 1.27 1.27)) hide)
+    )
+    (property "Datasheet" "" (at 192.405 89.535 0)
+      (effects (font (size 1.27 1.27)) hide)
+    )
+    (pin "1")
+    (instances
+      (project "Synth"
+        (path "/69caad27-d98a-4cdc-abd0-794bd5e6ba79/fff86bc7-37be-4dc8-9235-a859ce6d06d4"
+          (reference "#PWR05") (unit 1)
+        )
+      )
+    )
+  )
   (symbol (lib_id "Device:R") (at 120.65 105.41 0) (unit 1)
     (in_bom yes) (on_board yes) (dnp no) (fields_autoplaced)
@@
     )
   )
+  (symbol (lib_id "power:+12V") (at 192.405 74.295 0) (unit 1)
+    (in_bom yes) (on_board yes) (dnp no) (fields_autoplaced)
+    (property "Reference" "#PWR04" (at 192.405 78.105 0)
+      (effects (font (size 1.27 1.27)) hide)
+    )
+    (property "Value" "+12V" (at 192.405 69.85 0)
+      (effects (font (size 1.27 1.27)))
+    )
+    (property "Footprint" "" (at 192.405 74.295 0)
+      (effects (font (size 1.27 1.27)) hide)
+    )
+    (property "Datasheet" "" (at 192.405 74.295 0)
+      (effects (font (size 1.27 1.27)) hide)
+    )
+    (pin "1")
+    (instances
+      (project "Synth"
+        (path "/69caad27-d98a-4cdc-abd0-794bd5e6ba79/fff86bc7-37be-4dc8-9235-a859ce6d06d4"
+          (reference "#PWR04") (unit 1)
+        )
+      )
+    )
+  )
   (symbol (lib_id "Simulation_SPICE:NPN") (at 165.735 92.075 0) (unit 1)
     (in_bom yes) (on_board yes) (dnp no) (fields_autoplaced)
@@
         )
       )
+    )
+  )
+  (symbol (lib_id "power:+12V") (at 96.52 79.375 0) (unit 1)
+    (in_bom yes) (on_board yes) (dnp no) (fields_autoplaced)
+    (property "Reference" "#PWR03" (at 96.52 83.185 0)
+      (effects (font (size 1.27 1.27)) hide)
+    )
+    (property "Value" "+12V" (at 96.52 74.93 0)
+      (effects (font (size 1.27 1.27)))
+    )
+    (property "Footprint" "" (at 96.52 79.375 0)
+      (effects (font (size 1.27 1.27)) hide)
+    )
+    (property "Datasheet" "" (at 96.52 79.375 0)
+      (effects (font (size 1.27 1.27)) hide)
+    )
+    (pin "1")
+    (instances
+      (project "Synth"
+        (path "/69caad27-d98a-4cdc-abd0-794bd5e6ba79/fff86bc7-37be-4dc8-9235-a859ce6d06d4"
+          (reference "#PWR03") (unit 1)
+        )
+      )

Commit message: added some footprints
Parts:
- Q1, Q2, Q3, Q4: footprint (none) -> Package_TO_SOT_SMD:SOT-23-5_HandSoldering
- R10, R11, R12, R13, R14, R15, R16, R17, R18, R8, R9: footprint (none) -> Resistor_SMD:R_0805_2012Metric
Changed lines of the file:
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@@
       (effects (font (size 1.27 1.27)))
     )
-    (property "Footprint" "" (at 135.89 88.773 90)
+    (property "Footprint" "Resistor_SMD:R_0805_2012Metric" (at 135.89 88.773 90)
       (effects (font (size 1.27 1.27)) hide)
     )
@@
       (effects (font (size 1.27 1.27)))
     )
-    (property "Footprint" "" (at 183.515 86.233 90)
+    (property "Footprint" "Resistor_SMD:R_0805_2012Metric" (at 183.515 86.233 90)
       (effects (font (size 1.27 1.27)) hide)
     )
@@
       (effects (font (size 1.27 1.27)) (justify left))
     )
-    (property "Footprint" "" (at 153.67 80.645 0)
+    (property "Footprint" "Package_TO_SOT_SMD:SOT-23-5_HandSoldering" (at 153.67 80.645 0)
       (effects (font (size 1.27 1.27)) hide)
     )
@@
       (effects (font (size 1.27 1.27)) (justify left))
     )
-    (property "Footprint" "" (at 82.042 113.03 90)
+    (property "Footprint" "Resistor_SMD:R_0805_2012Metric" (at 82.042 113.03 90)
       (effects (font (size 1.27 1.27)) hide)
     )
@@
       (effects (font (size 1.27 1.27)))
     )
-    (property "Footprint" "" (at 192.405 67.183 90)
+    (property "Footprint" "Resistor_SMD:R_0805_2012Metric" (at 192.405 67.183 90)
       (effects (font (size 1.27 1.27)) hide)
     )
@@
       (effects (font (size 1.27 1.27)) (justify left))
     )
-    (property "Footprint" "" (at 201.295 78.105 0)
+    (property "Footprint" "Package_TO_SOT_SMD:SOT-23-5_HandSoldering" (at 201.295 78.105 0)
       (effects (font (size 1.27 1.27)) hide)
     )
@@
       (effects (font (size 1.27 1.27)) (justify left))
     )
-    (property "Footprint" "" (at 181.61 94.615 0)
+    (property "Footprint" "Package_TO_SOT_SMD:SOT-23-5_HandSoldering" (at 181.61 94.615 0)
       (effects (font (size 1.27 1.27)) hide)
     )
@@
       (effects (font (size 1.27 1.27)) (justify left))
     )
-    (property "Footprint" "" (at 118.872 105.41 90)
+    (property "Footprint" "Resistor_SMD:R_0805_2012Metric" (at 118.872 105.41 90)
       (effects (font (size 1.27 1.27)) hide)
     )
@@
       (effects (font (size 1.27 1.27)) (justify left))
     )
-    (property "Footprint" "" (at 229.235 92.075 0)
+    (property "Footprint" "Package_TO_SOT_SMD:SOT-23-5_HandSoldering" (at 229.235 92.075 0)
       (effects (font (size 1.27 1.27)) hide)
     )
@@
       (effects (font (size 1.27 1.27)) (justify left))
     )
-    (property "Footprint" "" (at 166.497 102.87 90)
+    (property "Footprint" "Resistor_SMD:R_0805_2012Metric" (at 166.497 102.87 90)
       (effects (font (size 1.27 1.27)) hide)
     )
@@
       (effects (font (size 1.27 1.27)))
     )
-    (property "Footprint" "" (at 72.39 96.393 90)
+    (property "Footprint" "Resistor_SMD:R_0805_2012Metric" (at 72.39 96.393 90)
       (effects (font (size 1.27 1.27)) hide)
     )
@@
       (effects (font (size 1.27 1.27)) (justify left))
     )
-    (property "Footprint" "" (at 118.872 71.755 90)
+    (property "Footprint" "Resistor_SMD:R_0805_2012Metric" (at 118.872 71.755 90)
       (effects (font (size 1.27 1.27)) hide)
     )
@@
       (effects (font (size 1.27 1.27)) (justify left))
     )
-    (property "Footprint" "" (at 166.497 69.215 90)
+    (property "Footprint" "Resistor_SMD:R_0805_2012Metric" (at 166.497 69.215 90)
       (effects (font (size 1.27 1.27)) hide)
     )
@@
       (effects (font (size 1.27 1.27)))
     )
-    (property "Footprint" "" (at 212.725 83.693 90)
+    (property "Footprint" "Resistor_SMD:R_0805_2012Metric" (at 212.725 83.693 90)
       (effects (font (size 1.27 1.27)) hide)
     )
@@
       (effects (font (size 1.27 1.27)))
     )
-    (property "Footprint" "" (at 144.78 69.723 90)
-      (effects (font (size 1.27 1.27)) hide)
-    )
+    (property "Footprint" "Resistor_SMD:R_0805_2012Metric" (at 144.78 69.723 90)
+      (effects (font (size 1.27 1.27)) hide)
+    )

Commit message: add the layout
Parts:
- RV4: footprint (none) -> Resistor_SMD:R_0805_2012Metric
Connections:
- net +12V: now also U4.5 (V+)
- net GND: now also U4.2 (V-)
Changed lines of the file:
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@@
+    )
+  )
+  (symbol (lib_id "power:GND") (at 144.78 92.075 0) (unit 1)
+    (in_bom yes) (on_board yes) (dnp no) (fields_autoplaced)
+    (property "Reference" "#PWR035" (at 144.78 98.425 0)
+      (effects (font (size 1.27 1.27)) hide)
+    )
+    (property "Value" "GND" (at 144.78 97.409 0)
+      (effects (font (size 1.27 1.27)))
+    )
+    (property "Footprint" "" (at 144.78 92.075 0)
+      (effects (font (size 1.27 1.27)) hide)
+    )
+    (property "Datasheet" "" (at 144.78 92.075 0)
+      (effects (font (size 1.27 1.27)) hide)
+    )
+    (pin "1")
+    (instances
+      (project "Synth"
+        (path "/69caad27-d98a-4cdc-abd0-794bd5e6ba79/fff86bc7-37be-4dc8-9235-a859ce6d06d4"
+          (reference "#PWR035") (unit 1)
+        )
+      )
     )
   )
@@
       (effects (font (size 1.27 1.27)) (justify right))
     )
-    (property "Footprint" "" (at 83.82 100.33 0)
+    (property "Footprint" "Resistor_SMD:R_0805_2012Metric" (at 83.82 100.33 0)
       (effects (font (size 1.27 1.27)) hide)
     )
@@
         )
       )
+    )
+  )
+  (symbol (lib_id "power:+12V") (at 144.78 76.835 0) (unit 1)
+    (in_bom yes) (on_board yes) (dnp no) (fields_autoplaced)
+    (property "Reference" "#PWR06" (at 144.78 80.645 0)
+      (effects (font (size 1.27 1.27)) hide)
+    )
+    (property "Value" "+12V" (at 144.78 72.39 0)
+      (effects (font (size 1.27 1.27)))
+    )
+    (property "Footprint" "" (at 144.78 76.835 0)
+      (effects (font (size 1.27 1.27)) hide)
+    )
+    (property "Datasheet" "" (at 144.78 76.835 0)
+      (effects (font (size 1.27 1.27)) hide)
+    )
+    (pin "1")
+    (instances
+      (project "Synth"
+        (path "/69caad27-d98a-4cdc-abd0-794bd5e6ba79/fff86bc7-37be-4dc8-9235-a859ce6d06d4"
+          (reference "#PWR06") (unit 1)
+        )
+      )

Commit message: fixed erc errs
Connections:
- net V_in+ renamed V_inW+
Changed lines of the file:
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@@
     (stroke (width 0) (type default))
   )
-  (global_label "V_in+" (shape input) (at 64.135 94.615 180) (fields_autoplaced)
+  (global_label "V_inW+" (shape input) (at 64.135 94.615 180) (fields_autoplaced)
     (effects (font (size 1.27 1.27)) (justify right))
-    (property "Intersheetrefs" "${INTERSHEET_REFS}" (at 55.7674 94.615 0)
+    (property "Intersheetrefs" "${INTERSHEET_REFS}" (at 54.316 94.615 0)
       (effects (font (size 1.27 1.27)) (justify right) hide)
     )

Commit message: changed the potentiometer footprints
Parts:
- RV4: footprint Resistor_SMD:R_0805_2012Metric -> Potentiometer_THT:Potentiometer_Bourns_3299W_Vertical
Changed lines of the file:
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@@
       (effects (font (size 1.27 1.27)) (justify right))
     )
-    (property "Footprint" "Resistor_SMD:R_0805_2012Metric" (at 83.82 100.33 0)
+    (property "Footprint" "Potentiometer_THT:Potentiometer_Bourns_3299W_Vertical" (at 83.82 100.33 0)
       (effects (font (size 1.27 1.27)) hide)
     )

Commit message: changed hierarchical labels
Connections:
- net V_Wavefolder+ renamed WF_out
Changed lines of the file:
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@@
     (stroke (width 0) (type default))
   )
-  (global_label "V_inW+" (shape input) (at 64.135 94.615 180) (fields_autoplaced)
+  (hierarchical_label "WF_out" (shape input) (at 222.25 81.915 0) (fields_autoplaced)
+    (effects (font (size 1.27 1.27)) (justify left))
+  )
+  (hierarchical_label "V_inW+" (shape input) (at 64.135 94.615 180) (fields_autoplaced)
     (effects (font (size 1.27 1.27)) (justify right))
-    (property "Intersheetrefs" "${INTERSHEET_REFS}" (at 54.316 94.615 0)
-      (effects (font (size 1.27 1.27)) (justify right) hide)
-    )
-  )
-  (global_label "V_Wavefolder+" (shape input) (at 222.25 81.915 0) (fields_autoplaced)
-    (effects (font (size 1.27 1.27)) (justify left))
-    (property "Intersheetrefs" "${INTERSHEET_REFS}" (at 239.0841 81.915 0)
-      (effects (font (size 1.27 1.27)) (justify left) hide)
-    )
   )
   (symbol (lib_id "Device:R") (at 135.89 86.995 90) (unit 1)
